File: kicad/08_lpddr4.kicad_sch (KiCad schematic)
At the start: 37 parts, among them U501 Ti135N484I3, U801 H9HCNNN8KUMLHR-NME

Commit message: Placement with power on the underside; LPDDR4 swizzle, 40/80 ohm rules, layer and plane plan
- LPDDR4 DQ swizzle within each byte (crossings 125 -> 45). efinity/pinplan/lpddr4_swizzle.json
  is the one source for the schematic (sheet 08) and the Interface Designer PIN_SWIZZLE_DQM*
  (read back and checked). Write-up in LPDDR4_SWIZZLE.md; scorer in tools/lpddr4_swizzle_score.py.
- Stack-up: a field solve (tools/zsolve.py) of JLC08161H-3313. Layer roles are now In1/In6 GND and
  In3/In4 planes, with signals on F/In2/In5/B. LPDDR4 widths follow the Efinix 40 ohm / 80 ohm
  guide (0.18 mm and 0.14/0.15 mm on In2/In5). Plane plan in TI135_PCB_NOTES.md section 6.6
  (KiCadRoutingTools recommend-stackup / recommend-plane-mappings).
- Ti135N484I3 LPDDR4 limit recorded: 2.8 Gbps (data sheet Table 22). Card-to-baseboard gap
  about 5.3 mm, so the power supplies go on the underside, as on the Ti60 card.
- Placement: the five TLV62585 cells are held to TI's Figure 24 layout (placement/sketches) and
  placed on B.Cu with J6's caps. J1/J2 are moved to the west edge, over an empty baseboard area.
  Seed 8 of 12 was applied: its quick route left 24 nets open, against 34 and 38 for the next
  seeds.
- LAYOUT_PLAN.md: the placement and routing plan, with the tool for each step.

Co-Authored-By: Claude Opus 5.5 <noreply@anthropic.com>
Connections:
- net ddr_dq0: now also U801.C4 (DQ6_A); no longer U801.B2 (DQ0_A)
- net ddr_dq1: now also U801.B4 (DQ7_A); no longer U801.C2 (DQ1_A)
- net ddr_dq10: now also U801.C9 (DQ14_A); no longer U801.E11 (DQ10_A)
- net ddr_dq11: now also U801.B9 (DQ15_A); no longer U801.F11 (DQ11_A)
- net ddr_dq12: now also U801.E11 (DQ10_A); no longer U801.F9 (DQ12_A)
- net ddr_dq13: now also U801.F11 (DQ11_A); no longer U801.E9 (DQ13_A)
- net ddr_dq14: now also U801.E9 (DQ13_A); no longer U801.C9 (DQ14_A)
- net ddr_dq15: now also U801.F9 (DQ12_A); no longer U801.B9 (DQ15_A)
- net ddr_dq16: now also U801.Y4 (DQ6_B); no longer U801.AA2 (DQ0_B)
- net ddr_dq17: now also U801.U2 (DQ3_B); no longer U801.Y2 (DQ1_B)
- net ddr_dq18: now also U801.AA4 (DQ7_B); no longer U801.V2 (DQ2_B)
- net ddr_dq19: now also U801.AA2 (DQ0_B); no longer U801.U2 (DQ3_B)
- net ddr_dq2: now also U801.B2 (DQ0_A); no longer U801.E2 (DQ2_A)
- net ddr_dq20: now also U801.Y2 (DQ1_B); no longer U801.U4 (DQ4_B)
- net ddr_dq21: now also U801.V2 (DQ2_B); no longer U801.V4 (DQ5_B)
- net ddr_dq22: now also U801.U4 (DQ4_B); no longer U801.Y4 (DQ6_B)
- net ddr_dq23: now also U801.V4 (DQ5_B); no longer U801.AA4 (DQ7_B)
- net ddr_dq24: now also U801.V9 (DQ13_B); no longer U801.AA11 (DQ8_B)
- net ddr_dq25: now also U801.AA9 (DQ15_B); no longer U801.Y11 (DQ9_B)
- net ddr_dq26: now also U801.Y9 (DQ14_B); no longer U801.V11 (DQ10_B)
- net ddr_dq27: now also U801.U9 (DQ12_B); no longer U801.U11 (DQ11_B)
- net ddr_dq28: now also U801.AA11 (DQ8_B); no longer U801.U9 (DQ12_B)
- net ddr_dq29: now also U801.Y11 (DQ9_B); no longer U801.V9 (DQ13_B)
- net ddr_dq3: now also U801.F4 (DQ4_A); no longer U801.F2 (DQ3_A)
- net ddr_dq30: now also U801.U11 (DQ11_B); no longer U801.Y9 (DQ14_B)
- net ddr_dq31: now also U801.V11 (DQ10_B); no longer U801.AA9 (DQ15_B)
- net ddr_dq4: now also U801.E4 (DQ5_A); no longer U801.F4 (DQ4_A)
- net ddr_dq5: now also U801.C2 (DQ1_A); no longer U801.E4 (DQ5_A)
- net ddr_dq6: now also U801.F2 (DQ3_A); no longer U801.C4 (DQ6_A)
- net ddr_dq7: now also U801.E2 (DQ2_A); no longer U801.B4 (DQ7_A)
Other:
- note added: "LPDDR4 x32: U501 DDR block -> U801 (2 channels x16, single rank). Wiring per TI135_PCB_NOTES.md §6.1 (Efinix Ti375C529 kit). DQ swizzled within each byte (LPDDR4_SWIZZLE.md, efinity/pinplan/lpddr4_swizzle.json, Interface Designer PIN_SWIZZLE_DQM0-3). Never DM/DQS/bytes/channels; CA not swizzled. Routing: §6.3 (40 R SE / 80 R diff, include package net lengths)."
- note removed: "LPDDR4 x32: U501 DDR block -> U801 (2 channels x16, single rank). Wiring per TI135_PCB_NOTES.md §6.1 (Efinix Ti375C529 kit). Swizzle rules §6.2: DQ only within its byte, CA only with the same permutation on both channels, never DM/DQS/bytes/channels; enter every swap in Interface Designer PIN_SWIZZLE_*. Routing: §6.3 (40 R SE / 80 R diff, include package net lengths)."
Changed lines of the file:
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@@
 		(comment 1 "Efinix Ti135N484I3 control card for the AC lab PSU baseboard")
 	)
-	(text "LPDDR4 x32: U501 DDR block -> U801 (2 channels x16, single rank). Wiring per TI135_PCB_NOTES.md §6.1\n(Efinix Ti375C529 kit). Swizzle rules §6.2: DQ only within its byte, CA only with the same permutation on\nboth channels, never DM/DQS/bytes/channels; enter every swap in Interface Designer PIN_SWIZZLE_*.\nRouting: §6.3 (40 R SE / 80 R diff, include package net lengths)."
+	(text "LPDDR4 x32: U501 DDR block -> U801 (2 channels x16, single rank). Wiring per TI135_PCB_NOTES.md §6.1\n(Efinix Ti375C529 kit). DQ swizzled within each byte (LPDDR4_SWIZZLE.md, efinity/pinplan/lpddr4_swizzle.json,\nInterface Designer PIN_SWIZZLE_DQM0-3). Never DM/DQS/bytes/channels; CA not swizzled.\nRouting: §6.3 (40 R SE / 80 R diff, include package net lengths)."
 		(exclude_from_sim no)
 		(at 17.78 20.32 0)
@@
 		)
 	)
-	(label "ddr_dq0"
+	(label "ddr_dq2"
 		(at 241.3 137.16 180)
 		(effects
@@
 		)
 	)
-	(label "ddr_dq7"
+	(label "ddr_dq1"
 		(at 241.3 154.94 180)
 		(effects
@@
 		)
 	)
-	(label "ddr_dq15"
+	(label "ddr_dq11"
 		(at 292.1 154.94 0)
 		(effects
@@
 		)
 	)
-	(label "ddr_dq1"
+	(label "ddr_dq5"
 		(at 241.3 139.7 180)
 		(effects
@@
 		)
 	)
-	(label "ddr_dq6"
+	(label "ddr_dq0"
 		(at 241.3 152.4 180)
 		(effects
@@
 		)
 	)
-	(label "ddr_dq14"
+	(label "ddr_dq10"
 		(at 292.1 152.4 0)
 		(effects
@@
 		)
 	)
-	(label "ddr_dq2"
+	(label "ddr_dq7"
 		(at 241.3 142.24 180)
 		(effects
@@
 		)
 	)
-	(label "ddr_dq5"
+	(label "ddr_dq4"
 		(at 241.3 149.86 180)
 		(effects
@@
 		)
 	)
-	(label "ddr_dq13"
+	(label "ddr_dq14"
 		(at 292.1 149.86 0)
 		(effects
@@
 		)
 	)
-	(label "ddr_dq10"
+	(label "ddr_dq12"
 		(at 292.1 142.24 0)
 		(effects
@@
 		)
 	)
-	(label "ddr_dq3"
+	(label "ddr_dq6"
 		(at 241.3 144.78 180)
 		(effects
@@
 		)
 	)
-	(label "ddr_dq4"
+	(label "ddr_dq3"
 		(at 241.3 147.32 180)
 		(effects
@@
 		)
 	)
-	(label "ddr_dq12"
+	(label "ddr_dq15"
 		(at 292.1 147.32 0)
 		(effects
@@
 		)
 	)
-	(label "ddr_dq11"
+	(label "ddr_dq13"
 		(at 292.1 144.78 0)
 		(effects
@@
 		)
 	)
-	(label "ddr_dq16"
+	(label "ddr_dq19"
 		(at 342.9 137.16 180)
 		(effects
@@
 		)
 	)
-	(label "ddr_dq23"
+	(label "ddr_dq18"
 		(at 342.9 154.94 180)
 		(effects
@@
 		)
 	)
-	(label "ddr_dq31"
+	(label "ddr_dq25"
 		(at 393.7 154.94 0)
 		(effects
@@
 		)
 	)
-	(label "ddr_dq24"
+	(label "ddr_dq28"
 		(at 393.7 137.16 0)
 		(effects
@@
 		)
 	)
-	(label "ddr_dq19"
+	(label "ddr_dq17"
 		(at 342.9 144.78 180)
 		(effects
@@
 		)
 	)
-	(label "ddr_dq20"
+	(label "ddr_dq22"
 		(at 342.9 147.32 180)
 		(effects
@@
 		)
 	)
-	(label "ddr_dq28"
+	(label "ddr_dq27"
 		(at 393.7 147.32 0)
 		(effects
@@
 		)
 	)
-	(label "ddr_dq27"
+	(label "ddr_dq30"
 		(at 393.7 144.78 0)
 		(effects
@@
 		)
 	)
-	(label "ddr_dq18"
+	(label "ddr_dq21"
 		(at 342.9 142.24 180)
 		(effects
@@
 		)
 	)
-	(label "ddr_dq21"
+	(label "ddr_dq23"
 		(at 342.9 149.86 180)
 		(effects
@@
 		)
 	)
-	(label "ddr_dq29"
+	(label "ddr_dq24"
 		(at 393.7 149.86 0)
 		(effects
@@
 		)
 	)
-	(label "ddr_dq26"
+	(label "ddr_dq31"
 		(at 393.7 142.24 0)
 		(effects
@@
 		)
 	)
-	(label "ddr_dq17"
+	(label "ddr_dq20"
 		(at 342.9 139.7 180)
 		(effects
@@
 		)
 	)
-	(label "ddr_dq22"
+	(label "ddr_dq16"
 		(at 342.9 152.4 180)
 		(effects
@@
 		)
 	)
-	(label "ddr_dq30"
+	(label "ddr_dq26"
 		(at 393.7 152.4 0)
 		(effects
@@
 		)
 	)
-	(label "ddr_dq25"
+	(label "ddr_dq29"
 		(at 393.7 139.7 0)
 		(effects

Commit message: Phase 3 (half): checklist fixes in the schematic; board placement still to do
- R801 240R 0.1 % (RT0402BRD07240RL, C852660); SSU_N (L4) 10 k pull-up R622 to 1V8.
- Efinix decoupling table in full on sheet 05 (now A2): C5001-C5073 (0201 10n/1n/100n,
  0402 1u/4u7, 0805 10u/47u, 1206 100u).
- Each TLV62585 cell: 47u output cap and a 22p feed-forward cap across R1 (data sheet:
  feed-forward needed above 47 uF; user decision).
- build_schematic.sh fails on duplicate references (ERC misses them).
- tools/add_parts.py: add missing schematic parts to a routed board; tools/place_free.py
  (untested): nearest free B.Cu spot.
- kicad/ti135_card.kicad_pcb unchanged; placement in work/p3, see NEXT_SESSION.md.

Co-Authored-By: Claude Opus 5.5 <noreply@anthropic.com>
Parts:
- R801: value 240R 1% -> 240R 0.1%; LCSC (none) -> C852660; MPN (none) -> RT0402BRD07240RL
Changed lines of the file:
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@@
 			)
 		)
-		(property "Value" "240R 1%"
-			(at 143.55 116.84 0)
+		(property "Value" "240R 0.1%"
+			(at 144.65 116.84 0)
 			(effects
 				(font
@@
 			(at 137.16 115.57 0)
 			(effects
+				(font
+					(size 1.27 1.27)
+				)
+				(hide yes)
+			)
+		)
+		(property "MPN" "RT0402BRD07240RL"
+			(at 137.16 115.57 0)
+			(effects
+				(font
+					(size 1.27 1.27)
+				)
+				(hide yes)
+			)
+		)
+		(property "LCSC" "C852660"
+			(at 137.16 115.57 0)
+			(effects
