File: kicad/08_lpddr4.kicad_sch (KiCad schematic)
At the start: 43 parts, among them U501 Ti135N484I3, U801 H9HCNNN8KUMLHR-NME

Commit message: R803 15 ohm: CKE peak 1376 mV at max/3200 (94 mV under the limit)
R803 (CKE series) 10R -> 15R, LCSC C25083. CKE rerun at typ/min/max on the
final routing: all corners pass; peak margin at max 208 mV at 2800 and
94 mV at 3200 (was 139 / 22 mV with 10 ohm).

Co-Authored-By: Claude Opus 5.5 <noreply@anthropic.com>
Parts:
- R803: value 10R -> 15R; LCSC C25077 -> C25083
Other:
- note added: "CKE series 15R on B.Cu at the U501 CKE via (sim/lpddr4_si/results/routed_corners.md): CKE has no ODT; without it the max-corner peak at 3200 Mbps is 1486 mV (limit 1470). Efinity has no CA/CKE drive setting."
- note removed: "CKE series 10R on B.Cu at the U501 CKE via (sim/lpddr4_si/results/routed_corners.md): CKE has no ODT; without it the max-corner peak at 3200 Mbps is 1486 mV (limit 1470), with it 1291 mV. Efinity has no CA/CKE drive setting."
Changed lines of the file:
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@@
 			)
 		)
-		(property "Value" "10R"
+		(property "Value" "15R"
 			(at 147.32 74.17 270)
 			(effects
@@
 			)
 		)
-		(property "LCSC" "C25077"
+		(property "LCSC" "C25083"
 			(at 147.32 76.2 0)
 			(effects
@@
 		)
 	)
-	(text "CKE series 10R on B.Cu at the U501 CKE via (sim/lpddr4_si/results/routed_corners.md):\nCKE has no ODT; without it the max-corner peak at 3200 Mbps is 1486 mV (limit 1470), with it 1291 mV.\nEfinity has no CA/CKE drive setting."
+	(text "CKE series 15R on B.Cu at the U501 CKE via (sim/lpddr4_si/results/routed_corners.md):\nCKE has no ODT; without it the max-corner peak at 3200 Mbps is 1486 mV (limit 1470).\nEfinity has no CA/CKE drive setting."
 		(exclude_from_sim no)
 		(at 127 66.04 0)

Commit message: 3D models for the BGAs (U501, U801, U1001, U601)
KiCad's library has no model for any of them (the footprints pointed at
missing STEP files), so tools/gen_bga_3d.py writes simple VRML models
(body, pin-1 dot, balls) to lib/3dmodels, from datasheet dimensions:
Efinix N484 model, SK hynix 200-ball FBGA, Kioxia P-WFBGA153, ISSI 24-ball
TFBGA (H). Linked as ${KIPRJMOD}/../lib/3dmodels so the CI render finds them.

U501 and U1001 footprints copied into ti135_card.pretty (footprint fields
updated on board, schematic, symbol lib); the U501 copy carries the board's
pad-to-die delays, which clears its lib_footprint_mismatch. DRC parity clean.

Co-Authored-By: Claude Opus 5.5 <noreply@anthropic.com>
Parts:
- U501: footprint Package_BGA:LFBGA-484_18x18mm_Layout22x22_P0.8mm -> ti135_card:LFBGA-484_18x18mm_Layout22x22_P0.8mm
Changed lines of the file:
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@@
 			)
 		)
-		(property "Footprint" "Package_BGA:LFBGA-484_18x18mm_Layout22x22_P0.8mm"
+		(property "Footprint" "ti135_card:LFBGA-484_18x18mm_Layout22x22_P0.8mm"
 			(at 88.9 139.7 0)
 			(hide yes)
