File: kicad/ti135_card.kicad_sch (KiCad schematic)
At the start: 0 parts

Commit message: Schematic complete: ethernet, emmc and adc sheets
- 09 ethernet: KSZ9031RNX with the Agilex 5 values and straps, RGMII 22R series,
  ferrite-fed analog rails, magjack J9, jack LED via 74LVC1G06
- 10 emmc: KIOXIA THGAMVG7T13BAIL, 47k pulls, CLK 10R, VCC 3V3 / VCCQ 1V8
- 13 adc: Agilex 3 card front end (SN74LV4051A, OPA365, 33R + 680p C0G,
  ADS7056 with DVDD 1V8), rail monitors on the mux
- attach/series_r/pull_r sheet helpers; STATUS.md updated

ERC: only the two known notes; all 92 pin-plan signals reach their loads.

Co-Authored-By: Claude Opus 5.5 <noreply@anthropic.com>
Other:
- sheet 09 ethernet ports: added eth_int_n, eth_mdc, eth_mdio, eth_rst_n, rgmii_rx_ctl, rgmii_rxc, rgmii_rxd0, rgmii_rxd1, rgmii_rxd2, rgmii_rxd3, rgmii_tx_ctl, rgmii_txc, rgmii_txd0, rgmii_txd1, rgmii_txd2, rgmii_txd3; removed none
- sheet 10 emmc ports: added emmc_clk, emmc_cmd, emmc_dat0, emmc_dat1, emmc_dat2, emmc_dat3, emmc_dat4, emmc_dat5, emmc_dat6, emmc_dat7, emmc_ds, emmc_rst_n; removed none
- sheet 13 adc ports: added adbsel0_3v3, adbsel1_3v3, adbsel2_3v3, adc_cs_n, adc_sclk, adc_sdo, isoada1, isoada2, isoada3; removed none

Commit message: Phase 3 (half): checklist fixes in the schematic; board placement still to do
- R801 240R 0.1 % (RT0402BRD07240RL, C852660); SSU_N (L4) 10 k pull-up R622 to 1V8.
- Efinix decoupling table in full on sheet 05 (now A2): C5001-C5073 (0201 10n/1n/100n,
  0402 1u/4u7, 0805 10u/47u, 1206 100u).
- Each TLV62585 cell: 47u output cap and a 22p feed-forward cap across R1 (data sheet:
  feed-forward needed above 47 uF; user decision).
- build_schematic.sh fails on duplicate references (ERC misses them).
- tools/add_parts.py: add missing schematic parts to a routed board; tools/place_free.py
  (untested): nearest free B.Cu spot.
- kicad/ti135_card.kicad_pcb unchanged; placement in work/p3, see NEXT_SESSION.md.

Co-Authored-By: Claude Opus 5.5 <noreply@anthropic.com>
Other:
- sheet 06 fpga_config ports: added fpga_ssu_n; removed none
- sheet 11 fpga_io ports: added fpga_ssu_n; removed none
