File: kicad/12_level_shift.kicad_sch (KiCad schematic)
At the start: 13 parts, among them U1201 SN74AXC8T245PWR, U1202 SN74AXC8T245PWR, U1203 SN74AXC8T245PWR, U1204 SN74AXC8T245PWR

Commit message: LCSC numbers for all JLC parts; Y701 -> YXC OT322525MJBA4SL
- tools/set_lcsc.py: one table (value, footprint) -> LCSC, fills empty LCSC fields in the
  sheets; 312 symbols. JLC basic parts where available, cap voltages checked per rail,
  VCORE divider 0.1 % (no 0.5 % in stock). Board fields synced with add_parts.py.
- Y701: the SiT8924 has no JLC stock; now YXC OT322525MJBA4SL (C669088, 3225), EN tied
  to 1V8. R701/C701 moved 0.5 mm to clear its courtyard. Netlist change: Y701 pin 1 -> 1V8.
- Only U501 (Ti135) is left without LCSC (global sourcing / consigned).
- DRC: schematic parity 0.

Co-Authored-By: Claude Opus 5.5 <noreply@anthropic.com>
Parts:
- C1201, C1202, C1203, C1204, C1205, C1206, C1207, C1208: LCSC (none) -> C1525
- R1201: LCSC (none) -> C25744
Changed lines of the file:
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@@
 			)
 		)
+		(property "LCSC" "C1525"
+			(at 320.04 127 0)
+			(effects
+				(font
+					(size 1.27 1.27)
+				)
+				(hide yes)
+			)
+		)
 		(pin "1"
 		)
@@
 			)
 		)
+		(property "LCSC" "C1525"
+			(at 144.78 48.26 0)
+			(effects
+				(font
+					(size 1.27 1.27)
+				)
+				(hide yes)
+			)
+		)
 		(pin "1"
 		)
@@
 			)
 		)
+		(property "LCSC" "C1525"
+			(at 144.78 127 0)
+			(effects
+				(font
+					(size 1.27 1.27)
+				)
+				(hide yes)
+			)
+		)
 		(pin "1"
 		)
@@
 			)
 		)
+		(property "LCSC" "C1525"
+			(at 309.88 48.26 0)
+			(effects
+				(font
+					(size 1.27 1.27)
+				)
+				(hide yes)
+			)
+		)
 		(pin "1"
 		)
@@
 			)
 		)
+		(property "LCSC" "C1525"
+			(at 154.94 48.26 0)
+			(effects
+				(font
+					(size 1.27 1.27)
+				)
+				(hide yes)
+			)
+		)
 		(pin "1"
 		)
@@
 			)
 		)
+		(property "LCSC" "C1525"
+			(at 154.94 127 0)
+			(effects
+				(font
+					(size 1.27 1.27)
+				)
+				(hide yes)
+			)
+		)
 		(pin "1"
 		)
@@
 			)
 		)
+		(property "LCSC" "C25744"
+			(at 38.1 45.72 0)
+			(effects
+				(font
+					(size 1.27 1.27)
+				)
+				(hide yes)
+			)
+		)
 		(pin "1"
 		)
@@
 			)
 		)
+		(property "LCSC" "C1525"
+			(at 320.04 48.26 0)
+			(effects
+				(font
+					(size 1.27 1.27)
+				)
+				(hide yes)
+			)
+		)
 		(pin "1"
 		)
@@
 			)
 		)
+		(property "LCSC" "C1525"
+			(at 309.88 127 0)
+			(effects
+				(font
+					(size 1.27 1.27)
+				)
+				(hide yes)
+			)
+		)
