File: kicad/14_connectors.kicad_sch (KiCad schematic)
At the start: 13 parts, among them J2 UART 3.3V, J3 2x19 1.27mm socket (bottom), J5 LCD 1x14 2.54mm

Commit message: J101 bench 5 V header, J3 0.9/0.6 mm pads, baseboard U8 2 A
- J101 (sheet 01): 2.54 mm 1x2 header on F.Cu north-east of J6, pin 1 5V0 / pin 2 GND,
  to power the card with female jumpers without the baseboard. On the 5V0 B.Cu pour and
  the GND planes; nothing on the baseboard under its tails (MECHANICAL.md).
- J3: project-local footprint ti135_card:PinSocket_2x19_P1.27mm_Vertical_Drill0.6
  (pads 0.9 mm, drill 0.6 mm, as on the Agilex card) so a 0.1 mm track fits between pins.
- Baseboard U8 is now the Mornsun K7805-2000R3 (5 V / 2 A; ac_psu_kicad 732c9b1):
  POWER_BUDGET, STATUS and MECHANICAL updated; 20V_ISO_SEC still to be measured.
- Board: also the routing in progress. DRC: schematic parity 0.

Co-Authored-By: Claude Opus 5.5 <noreply@anthropic.com>
Parts:
- J3: footprint Connector_PinSocket_1.27mm:PinSocket_2x19_P1.27mm_Vertical -> ti135_card:PinSocket_2x19_P1.27mm_Vertical_Drill0.6
Changed lines of the file:
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@@
 			)
 		)
-		(property "Footprint" "Connector_PinSocket_1.27mm:PinSocket_2x19_P1.27mm_Vertical"
+		(property "Footprint" "ti135_card:PinSocket_2x19_P1.27mm_Vertical_Drill0.6"
 			(at 88.9 43.18 0)
 			(hide yes)

Commit message: LCSC numbers for all JLC parts; Y701 -> YXC OT322525MJBA4SL
- tools/set_lcsc.py: one table (value, footprint) -> LCSC, fills empty LCSC fields in the
  sheets; 312 symbols. JLC basic parts where available, cap voltages checked per rail,
  VCORE divider 0.1 % (no 0.5 % in stock). Board fields synced with add_parts.py.
- Y701: the SiT8924 has no JLC stock; now YXC OT322525MJBA4SL (C669088, 3225), EN tied
  to 1V8. R701/C701 moved 0.5 mm to clear its courtyard. Netlist change: Y701 pin 1 -> 1V8.
- Only U501 (Ti135) is left without LCSC (global sourcing / consigned).
- DRC: schematic parity 0.

Co-Authored-By: Claude Opus 5.5 <noreply@anthropic.com>
Parts:
- J2: LCSC (none) -> C2937625
- J3: LCSC (none) -> C27985219
- J5: LCSC (none) -> C22465874
- R1401, R1402: LCSC (none) -> C11702
Changed lines of the file:
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@@
+			)
+		)
+		(property "LCSC" "C11702"
+			(at 167.64 175.26 0)
+			(effects
+				(font
+					(size 1.27 1.27)
+				)
+				(hide yes)
 			)
 		)
@@
 			)
 		)
+		(property "LCSC" "C27985219"
+			(at 88.9 43.18 0)
+			(effects
+				(font
+					(size 1.27 1.27)
+				)
+				(hide yes)
+			)
+		)
 		(pin "1"
 		)
@@
 			)
 		)
+		(property "LCSC" "C11702"
+			(at 167.64 177.8 0)
+			(effects
+				(font
+					(size 1.27 1.27)
+				)
+				(hide yes)
+			)
+		)
 		(pin "1"
 		)
@@
 			)
 		)
+		(property "LCSC" "C2937625"
+			(at 190.5 177.8 0)
+			(effects
+				(font
+					(size 1.27 1.27)
+				)
+				(hide yes)
+			)
+		)
 		(pin "1"
 		)
@@
 			)
 		)
+		(property "LCSC" "C22465874"
+			(at 76.2 152.4 0)
+			(effects
+				(font
+					(size 1.27 1.27)
+				)
+				(hide yes)
+			)
+		)
