File: kicad/07_clocks.kicad_sch (KiCad schematic)
At the start: 5 parts, among them Y701 SiT8924BA-73-18N-25.000000

Commit message: LCSC numbers for all JLC parts; Y701 -> YXC OT322525MJBA4SL
- tools/set_lcsc.py: one table (value, footprint) -> LCSC, fills empty LCSC fields in the
  sheets; 312 symbols. JLC basic parts where available, cap voltages checked per rail,
  VCORE divider 0.1 % (no 0.5 % in stock). Board fields synced with add_parts.py.
- Y701: the SiT8924 has no JLC stock; now YXC OT322525MJBA4SL (C669088, 3225), EN tied
  to 1V8. R701/C701 moved 0.5 mm to clear its courtyard. Netlist change: Y701 pin 1 -> 1V8.
- Only U501 (Ti135) is left without LCSC (global sourcing / consigned).
- DRC: schematic parity 0.

Co-Authored-By: Claude Opus 5.5 <noreply@anthropic.com>
Parts:
- C701: LCSC (none) -> C1525
- R701, R702, R703: LCSC (none) -> C25105
- Y701: value SiT8924BA-73-18N-25.000000 -> OT322525MJBA4SL; footprint Oscillator:Oscillator_SMD_SiT_PQFN-4Pin_2.0x1.6mm -> Oscillator:Oscillator_SMD_Abracon_ASE-4Pin_3.2x2.5mm; symbol ti135_card:SIT8924BA-73-18N-25.000000 -> ti135_card:OT322525MJBA4SL; LCSC (none) -> C669088
Connections:
- net 1V8: now also Y701.1 (EN)
- no-connect marks 1 -> 0
Other:
- note added: "Y701 EN (pin 1) tied to 1V8: always enabled."
Changed lines of the file:
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@@
 		(color 0 0 0 0)
-	)
-	(no_connect
-		(at 68.58 63.5)
 	)
 	(wire
@@
 			)
 		)
+		(property "LCSC" "C1525"
+			(at 50.8 57.15 0)
+			(effects
+				(font
+					(size 1.27 1.27)
+				)
+				(hide yes)
+			)
+		)
 		(pin "1"
 		)
@@
 			)
 		)
+		(property "LCSC" "C25105"
+			(at 104.14 63.5 0)
+			(effects
+				(font
+					(size 1.27 1.27)
+				)
+				(hide yes)
+			)
+		)
 		(pin "1"
 		)
@@
 			)
 		)
+		(property "LCSC" "C25105"
+			(at 104.14 73.66 0)
+			(effects
+				(font
+					(size 1.27 1.27)
+				)
+				(hide yes)
+			)
+		)
 		(pin "1"
 		)
@@
 	)
 	(symbol
-		(lib_id "ti135_card:SIT8924BA-73-18N-25.000000")
+		(lib_id "ti135_card:OT322525MJBA4SL")
 		(at 76.2 63.5 0)
 		(unit 1)
@@
 			)
 		)
-		(property "Value" "SiT8924BA-73-18N-25.000000"
+		(property "Value" "OT322525MJBA4SL"
 			(at 77.47 69.85 0)
 			(show_name no)
@@
 			)
 		)
-		(property "Footprint" "Oscillator:Oscillator_SMD_SiT_PQFN-4Pin_2.0x1.6mm"
+		(property "Footprint" "Oscillator:Oscillator_SMD_Abracon_ASE-4Pin_3.2x2.5mm"
 			(at 93.98 72.39 0)
 			(hide yes)
@@
 					(size 1.27 1.27)
 				)
+			)
+		)
+		(property "LCSC" "C669088"
+			(at 76.2 63.5 0)
+			(effects
+				(font
+					(size 1.27 1.27)
+				)
+				(hide yes)
 			)
 		)
@@
 			)
 		)
+		(property "LCSC" "C25105"
+			(at 104.14 53.34 0)
+			(effects
+				(font
+					(size 1.27 1.27)
+				)
+				(hide yes)
+			)
+		)
 		(pin "1"
 		)
@@
 		)
 	)
+	(wire
+		(pts
+			(xy 68.58 63.5) (xy 66.04 63.5)
+		)
+		(stroke
+			(width 0)
+			(type default)
+		)
+	)
+	(wire
+		(pts
+			(xy 66.04 63.5) (xy 66.04 59.69)
+		)
+		(stroke
+			(width 0)
+			(type default)
+		)
+	)
+	(symbol
+		(lib_id "ti135_card:1V8")
+		(at 66.04 59.69 0)
+		(unit 1)
+		(exclude_from_sim no)
+		(in_bom yes)
+		(on_board yes)
+		(dnp no)
+		(property "Reference" "#PWR07005"
+			(at 66.04 63.5 0)
+			(effects
+				(font
+					(size 1.27 1.27)
+				)
+				(hide yes)
+			)
+		)
+		(property "Value" "1V8"
+			(at 66.04 56.134 0)
+			(effects
+				(font
+					(size 1.27 1.27)
+				)
+			)
+		)
+		(property "Footprint" ""
+			(at 66.04 59.69 0)
+			(effects
+				(font
+					(size 1.27 1.27)
+				)
+				(hide yes)
+			)
+		)
+		(property "Datasheet" ""
+			(at 66.04 59.69 0)
+			(effects
+				(font
+					(size 1.27 1.27)
+				)
+				(hide yes)
+			)
+		)
+		(property "Description" "Power symbol for net \"1V8\" (IPC net name)"
+			(at 66.04 59.69 0)
+			(effects
+				(font
+					(size 1.27 1.27)
+				)
+				(hide yes)
+			)
+		)
+		(pin "1"
+		)
+		(instances
+			(project "ti135_card"
+				(path "/c384d3ae-6e7d-47ca-8f4d-7f9f77efe4b7/8a939fee-b0ba-4a20-ad16-1502b11e2d82"
+					(reference "#PWR07005")
+					(unit 1)
+				)
+			)
+		)
+	)
+	(text "Y701 EN (pin 1) tied to 1V8: always enabled."
+		(exclude_from_sim no)
+		(at 63.5 76.2 0)
+		(effects
+			(font
+				(size 1.27 1.27)
+			)
+			(justify left bottom)
+		)
+	)

Commit message: Y701: SiT PQFN 3.2x2.5 footprint (matches the YXC land pattern)
YXC YSO110TR data sheet (OT322525MJBA4SL), 3225 recommended pattern: pads 1.3 x 1.2,
gaps 0.8 / 0.7 mm. Oscillator_SMD_SiT_PQFN-4Pin_3.2x2.5mm has the same gaps and pad
height (pads 1.4 x 1.2); the Abracon ASE one had a 0.55 mm gap and 1.1 mm pads.
Data sheet also confirms pin 1 tri-state: high or floating = enabled (EN tied to 1V8).
J3 HC-PM127-4.3H-2x19PZ drawing: 0.45 x 0.15 pins, recommended hole 0.6 mm (as J3 now).

Co-Authored-By: Claude Opus 5.5 <noreply@anthropic.com>
Parts:
- Y701: footprint Oscillator:Oscillator_SMD_Abracon_ASE-4Pin_3.2x2.5mm -> Oscillator:Oscillator_SMD_SiT_PQFN-4Pin_3.2x2.5mm
Changed lines of the file:
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@@
 			)
 		)
-		(property "Footprint" "Oscillator:Oscillator_SMD_Abracon_ASE-4Pin_3.2x2.5mm"
+		(property "Footprint" "Oscillator:Oscillator_SMD_SiT_PQFN-4Pin_3.2x2.5mm"
 			(at 93.98 72.39 0)
 			(hide yes)
