File: kicad/06_fpga_config.kicad_sch (KiCad schematic)
At the start: 26 parts, among them J1 JTAG 3.3V, U501 Ti135N484I3, U601 IS25WP128-RHLE

Commit message: Phase 3 (half): checklist fixes in the schematic; board placement still to do
- R801 240R 0.1 % (RT0402BRD07240RL, C852660); SSU_N (L4) 10 k pull-up R622 to 1V8.
- Efinix decoupling table in full on sheet 05 (now A2): C5001-C5073 (0201 10n/1n/100n,
  0402 1u/4u7, 0805 10u/47u, 1206 100u).
- Each TLV62585 cell: 47u output cap and a 22p feed-forward cap across R1 (data sheet:
  feed-forward needed above 47 uF; user decision).
- build_schematic.sh fails on duplicate references (ERC misses them).
- tools/add_parts.py: add missing schematic parts to a routed board; tools/place_free.py
  (untested): nearest free B.Cu spot.
- kicad/ti135_card.kicad_pcb unchanged; placement in work/p3, see NEXT_SESSION.md.

Co-Authored-By: Claude Opus 5.5 <noreply@anthropic.com>
Parts:
- added R622: 10k, Resistor_SMD:R_0402_1005Metric, symbol ti135_card:R
Connections:
- net 1V8: now also R622.1
- new net fpga_ssu_n: R622.2
Other:
- note added: "SSU_N: weak pull-up (checklist)"
Changed lines of the file:
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@@
+		)
+	)
+	(hierarchical_label "fpga_ssu_n"
+		(shape passive)
+		(at 177.8 195.58 270)
+		(effects
+			(font
+				(size 1.27 1.27)
+			)
+			(justify right)
+		)
+	)
+	(wire
+		(pts
+			(xy 177.8 195.58) (xy 177.8 193.04)
+		)
+		(stroke
+			(width 0)
+			(type default)
+		)
+	)
+	(label "fpga_ssu_n"
+		(at 177.8 193.04 90)
+		(effects
+			(font
+				(size 1.27 1.27)
+			)
+			(justify left bottom)
+		)
+	)
+	(symbol
+		(lib_id "ti135_card:R")
+		(at 190.5 177.8 0)
+		(unit 1)
+		(exclude_from_sim no)
+		(in_bom yes)
+		(on_board yes)
+		(dnp no)
+		(property "Reference" "R622"
+			(at 195.24 176.53 0)
+			(effects
+				(font
+					(size 1.27 1.27)
+				)
+			)
+		)
+		(property "Value" "10k"
+			(at 194.69 179.07 0)
+			(effects
+				(font
+					(size 1.27 1.27)
+				)
+			)
+		)
+		(property "Footprint" "Resistor_SMD:R_0402_1005Metric"
+			(at 188.722 177.8 0)
+			(effects
+				(font
+					(size 1.27 1.27)
+				)
+				(hide yes)
+			)
+		)
+		(property "Datasheet" ""
+			(at 190.5 177.8 0)
+			(effects
+				(font
+					(size 1.27 1.27)
+				)
+				(hide yes)
+			)
+		)
+		(property "Description" "Resistor"
+			(at 190.5 177.8 0)
+			(effects
+				(font
+					(size 1.27 1.27)
+				)
+				(hide yes)
+			)
+		)
+		(pin "1"
+		)
+		(pin "2"
+		)
+		(instances
+			(project "ti135_card"
+				(path "/c384d3ae-6e7d-47ca-8f4d-7f9f77efe4b7/005bb34e-5019-4cde-82e0-1ce10912d4b9"
+					(reference "R622")
+					(unit 1)
+				)
+			)
+		)
+	)
+	(wire
+		(pts
+			(xy 190.5 173.99) (xy 190.5 171.45)
+		)
+		(stroke
+			(width 0)
+			(type default)
+		)
+	)
+	(symbol
+		(lib_id "ti135_card:1V8")
+		(at 190.5 171.45 0)
+		(unit 1)
+		(exclude_from_sim no)
+		(in_bom yes)
+		(on_board yes)
+		(dnp no)
+		(property "Reference" "#PWR027"
+			(at 190.5 175.26 0)
+			(effects
+				(font
+					(size 1.27 1.27)
+				)
+				(hide yes)
+			)
+		)
+		(property "Value" "1V8"
+			(at 190.5 167.894 0)
+			(effects
+				(font
+					(size 1.27 1.27)
+				)
+			)
+		)
+		(property "Footprint" ""
+			(at 190.5 171.45 0)
+			(effects
+				(font
+					(size 1.27 1.27)
+				)
+				(hide yes)
+			)
+		)
+		(property "Datasheet" ""
+			(at 190.5 171.45 0)
+			(effects
+				(font
+					(size 1.27 1.27)
+				)
+				(hide yes)
+			)
+		)
+		(property "Description" "Power symbol for net \"1V8\" (IPC net name)"
+			(at 190.5 171.45 0)
+			(effects
+				(font
+					(size 1.27 1.27)
+				)
+				(hide yes)
+			)
+		)
+		(pin "1"
+		)
+		(instances
+			(project "ti135_card"
+				(path "/c384d3ae-6e7d-47ca-8f4d-7f9f77efe4b7/005bb34e-5019-4cde-82e0-1ce10912d4b9"
+					(reference "#PWR027")
+					(unit 1)
+				)
+			)
+		)
+	)
+	(wire
+		(pts
+			(xy 190.5 181.61) (xy 190.5 184.15)
+		)
+		(stroke
+			(width 0)
+			(type default)
+		)
+	)
+	(label "fpga_ssu_n"
+		(at 190.5 184.15 270)
+		(effects
+			(font
+				(size 1.27 1.27)
+			)
+			(justify right bottom)
+		)
+	)
+	(text "SSU_N: weak pull-up (checklist)"
+		(exclude_from_sim no)
+		(at 170.18 162.56 0)
+		(effects
+			(font
+				(size 1.27 1.27)
+			)
+			(justify left bottom)
 		)
 	)

Commit message: LCSC numbers for all JLC parts; Y701 -> YXC OT322525MJBA4SL
- tools/set_lcsc.py: one table (value, footprint) -> LCSC, fills empty LCSC fields in the
  sheets; 312 symbols. JLC basic parts where available, cap voltages checked per rail,
  VCORE divider 0.1 % (no 0.5 % in stock). Board fields synced with add_parts.py.
- Y701: the SiT8924 has no JLC stock; now YXC OT322525MJBA4SL (C669088, 3225), EN tied
  to 1V8. R701/C701 moved 0.5 mm to clear its courtyard. Netlist change: Y701 pin 1 -> 1V8.
- Only U501 (Ti135) is left without LCSC (global sourcing / consigned).
- DRC: schematic parity 0.

Co-Authored-By: Claude Opus 5.5 <noreply@anthropic.com>
Parts:
- C615: LCSC (none) -> C1525
- D601, D602: LCSC (none) -> C2286
- J1: LCSC (none) -> C492404
- R601, R602, R603, R604, R605, R606, R607, R608, R609, R610, R611, R612, R613, R614, R616, R617, R618, R619, R622: LCSC (none) -> C25744
- R620, R621: LCSC (none) -> C11702
Changed lines of the file:
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@@
 			)
 		)
+		(property "LCSC" "C25744"
+			(at 50.8 127 0)
+			(effects
+				(font
+					(size 1.27 1.27)
+				)
+				(hide yes)
+			)
+		)
 		(pin "1"
 		)
@@
 			)
 		)
+		(property "LCSC" "C25744"
+			(at 38.1 127 0)
+			(effects
+				(font
+					(size 1.27 1.27)
+				)
+				(hide yes)
+			)
+		)
 		(pin "1"
 		)
@@
 			)
 		)
+		(property "LCSC" "C25744"
+			(at 63.5 127 0)
+			(effects
+				(font
+					(size 1.27 1.27)
+				)
+				(hide yes)
+			)
+		)
 		(pin "1"
 		)
@@
 			)
 		)
+		(property "LCSC" "C25744"
+			(at 167.64 86.36 0)
+			(effects
+				(font
+					(size 1.27 1.27)
+				)
+				(hide yes)
+			)
+		)
 		(pin "1"
 		)
@@
 			)
 		)
+		(property "LCSC" "C2286"
+			(at 335.28 187.96 0)
+			(effects
+				(font
+					(size 1.27 1.27)
+				)
+				(hide yes)
+			)
+		)
 		(pin "1"
 		)
@@
 			)
 		)
+		(property "LCSC" "C25744"
+			(at 266.7 119.38 0)
+			(effects
+				(font
+					(size 1.27 1.27)
+				)
+				(hide yes)
+			)
+		)
 		(pin "1"
 		)
@@
 			)
 		)
+		(property "LCSC" "C25744"
+			(at 76.2 127 0)
+			(effects
+				(font
+					(size 1.27 1.27)
+				)
+				(hide yes)
+			)
+		)
 		(pin "1"
 		)
@@
 			)
 		)
+		(property "LCSC" "C2286"
+			(at 317.5 187.96 0)
+			(effects
+				(font
+					(size 1.27 1.27)
+				)
+				(hide yes)
+			)
+		)
 		(pin "1"
 		)
@@
 			)
 		)
+		(property "LCSC" "C25744"
+			(at 179.07 86.36 0)
+			(effects
+				(font
+					(size 1.27 1.27)
+				)
+				(hide yes)
+			)
+		)
 		(pin "1"
 		)
@@
 			)
 		)
+		(property "LCSC" "C492404"
+			(at 152.4 139.7 0)
+			(effects
+				(font
+					(size 1.27 1.27)
+				)
+				(hide yes)
+			)
+		)
 		(pin "1"
 		)
@@
 			)
 		)
+		(property "LCSC" "C25744"
+			(at 279.4 119.38 0)
+			(effects
+				(font
+					(size 1.27 1.27)
+				)
+				(hide yes)
+			)
+		)
 		(pin "1"
 		)
@@
 			)
 		)
+		(property "LCSC" "C25744"
+			(at 88.9 127 0)
+			(effects
+				(font
+					(size 1.27 1.27)
+				)
+				(hide yes)
+			)
+		)
 		(pin "1"
 		)
@@
 			)
 		)
+		(property "LCSC" "C25744"
+			(at 127 177.8 0)
+			(effects
+				(font
+					(size 1.27 1.27)
+				)
+				(hide yes)
+			)
+		)
 		(pin "1"
 		)
@@
 			)
 		)
+		(property "LCSC" "C25744"
+			(at 139.7 177.8 0)
+			(effects
+				(font
+					(size 1.27 1.27)
+				)
+				(hide yes)
+			)
+		)
 		(pin "1"
 		)
@@
 			)
 		)
+		(property "LCSC" "C25744"
+			(at 304.8 119.38 0)
+			(effects
+				(font
+					(size 1.27 1.27)
+				)
+				(hide yes)
+			)
+		)
 		(pin "1"
 		)
@@
 			)
 		)
+		(property "LCSC" "C25744"
+			(at 190.5 86.36 0)
+			(effects
+				(font
+					(size 1.27 1.27)
+				)
+				(hide yes)
+			)
+		)
 		(pin "1"
 		)
@@
 			)
 		)
+		(property "LCSC" "C25744"
+			(at 114.3 177.8 0)
+			(effects
+				(font
+					(size 1.27 1.27)
+				)
+				(hide yes)
+			)
+		)
 		(pin "1"
 		)
@@
 			)
 		)
+		(property "LCSC" "C11702"
+			(at 335.28 177.8 0)
+			(effects
+				(font
+					(size 1.27 1.27)
+				)
+				(hide yes)
+			)
+		)
 		(pin "1"
 		)
@@
 			)
 		)
+		(property "LCSC" "C25744"
+			(at 292.1 119.38 0)
+			(effects
+				(font
+					(size 1.27 1.27)
+				)
+				(hide yes)
+			)
+		)
 		(pin "1"
 		)
@@
 			)
 		)
+		(property "LCSC" "C25744"
+			(at 101.6 127 0)
+			(effects
+				(font
+					(size 1.27 1.27)
+				)
+				(hide yes)
+			)
+		)
 		(pin "1"
 		)
@@
 			)
 		)
+		(property "LCSC" "C25744"
+			(at 101.6 177.8 0)
+			(effects
+				(font
+					(size 1.27 1.27)
+				)
+				(hide yes)
+			)
+		)
 		(pin "1"
 		)
@@
 			)
 		)
+		(property "LCSC" "C25744"
+			(at 201.93 86.36 0)
+			(effects
+				(font
+					(size 1.27 1.27)
+				)
+				(hide yes)
+			)
+		)
 		(pin "1"
 		)
@@
 			)
 		)
+		(property "LCSC" "C25744"
+			(at 190.5 177.8 0)
+			(effects
+				(font
+					(size 1.27 1.27)
+				)
+				(hide yes)
+			)
+		)
 		(pin "1"
 		)
@@
 			)
 		)
+		(property "LCSC" "C1525"
+			(at 342.9 71.12 0)
+			(effects
+				(font
+					(size 1.27 1.27)
+				)
+				(hide yes)
+			)
+		)
 		(pin "1"
 		)
@@
 			)
 		)
+		(property "LCSC" "C11702"
+			(at 317.5 177.8 0)
+			(effects
+				(font
+					(size 1.27 1.27)
+				)
+				(hide yes)
+			)
+		)

Commit message: 3D models for the BGAs (U501, U801, U1001, U601)
KiCad's library has no model for any of them (the footprints pointed at
missing STEP files), so tools/gen_bga_3d.py writes simple VRML models
(body, pin-1 dot, balls) to lib/3dmodels, from datasheet dimensions:
Efinix N484 model, SK hynix 200-ball FBGA, Kioxia P-WFBGA153, ISSI 24-ball
TFBGA (H). Linked as ${KIPRJMOD}/../lib/3dmodels so the CI render finds them.

U501 and U1001 footprints copied into ti135_card.pretty (footprint fields
updated on board, schematic, symbol lib); the U501 copy carries the board's
pad-to-die delays, which clears its lib_footprint_mismatch. DRC parity clean.

Co-Authored-By: Claude Opus 5.5 <noreply@anthropic.com>
Parts:
- U501: footprint Package_BGA:LFBGA-484_18x18mm_Layout22x22_P0.8mm -> ti135_card:LFBGA-484_18x18mm_Layout22x22_P0.8mm
Changed lines of the file:
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@@
 			)
 		)
-		(property "Footprint" "Package_BGA:LFBGA-484_18x18mm_Layout22x22_P0.8mm"
+		(property "Footprint" "ti135_card:LFBGA-484_18x18mm_Layout22x22_P0.8mm"
 			(at 139.7 76.2 0)
 			(hide yes)
