File: kicad/10_emmc.kicad_sch (KiCad schematic)
At the start: 0 parts

Commit message: Schematic complete: ethernet, emmc and adc sheets
- 09 ethernet: KSZ9031RNX with the Agilex 5 values and straps, RGMII 22R series,
  ferrite-fed analog rails, magjack J9, jack LED via 74LVC1G06
- 10 emmc: KIOXIA THGAMVG7T13BAIL, 47k pulls, CLK 10R, VCC 3V3 / VCCQ 1V8
- 13 adc: Agilex 3 card front end (SN74LV4051A, OPA365, 33R + 680p C0G,
  ADS7056 with DVDD 1V8), rail monitors on the mux
- attach/series_r/pull_r sheet helpers; STATUS.md updated

ERC: only the two known notes; all 92 pin-plan signals reach their loads.

Co-Authored-By: Claude Opus 5.5 <noreply@anthropic.com>
Parts:
- added C1001, C1004: 4u7, Capacitor_SMD:C_0402_1005Metric, symbol ti135_card:C
- added C1002, C1003, C1005, C1006: 100n, Capacitor_SMD:C_0402_1005Metric, symbol ti135_card:C
- added C1007: 2u2, Capacitor_SMD:C_0402_1005Metric, symbol ti135_card:C
- added R1001: 10R, Resistor_SMD:R_0402_1005Metric, symbol ti135_card:R
- added R1010, R1011, R1012, R1013, R1014, R1015, R1016, R1017, R1018, R1019, R1020: 47k, Resistor_SMD:R_0402_1005Metric, symbol ti135_card:R
- added U1001: THGAMVG7T13BAIL, Package_BGA:LFBGA-153_11.5x13mm_Layout14x14_P0.5mm, symbol ti135_card:THGAMVG7T13BAIL
Connections:
- new net 1V8: C1004.1, C1005.1, C1006.1, R1010.1, R1011.1, R1012.1, R1013.1, R1014.1, R1015.1, R1016.1, R1017.1, R1018.1, R1019.1, U1001.C6 (VCCQ), U1001.M4 (VCCQ), U1001.N4 (VCCQ), U1001.P3 (VCCQ), U1001.P5 (VCCQ)
- new net 3V3: C1001.1, C1002.1, C1003.1, U1001.E6 (VCC), U1001.F5 (VCC), U1001.J10 (VCC), U1001.K9 (VCC)
- new net GND: C1001.2, C1002.2, C1003.2, C1004.2, C1005.2, C1006.2, C1007.2, R1020.2, U1001.A6 (VSS), U1001.C4 (VSSQ), U1001.E7 (VSS), U1001.G5 (VSS), U1001.H10 (VSS), U1001.J5 (VSS), U1001.K8 (VSS), U1001.N2 (VSSQ), U1001.N5 (VSSQ), U1001.P4 (VSSQ), U1001.P6 (VSSQ)
- new net emmc_clk: R1001.1
- new net emmc_clk_r: R1001.2, U1001.M6 (CLK)
- new net emmc_cmd: R1010.2, U1001.M5 (CMD)
- new net emmc_dat0: R1011.2, U1001.A3 (DAT0)
- new net emmc_dat1: R1012.2, U1001.A4 (DAT1)
- new net emmc_dat2: R1013.2, U1001.A5 (DAT2)
- new net emmc_dat3: R1014.2, U1001.B2 (DAT3)
- new net emmc_dat4: R1015.2, U1001.B3 (DAT4)
- new net emmc_dat5: R1016.2, U1001.B4 (DAT5)
- new net emmc_dat6: R1017.2, U1001.B5 (DAT6)
- new net emmc_dat7: R1018.2, U1001.B6 (DAT7)
- new net emmc_ds: R1020.1, U1001.H5 (DS)
- new net emmc_rst_n: R1019.2, U1001.K5 (RST_n)
- new net emmc_vddi: C1007.1, U1001.C2 (VDDi)
Other:
- note added: "Pull-ups 47 k to 1V8 (CMD, DAT0-7, RST_n); DS 47 k pull-down"
- note added: "VCC 3V3: 4u7 + 2 x 100n"
- note added: "VCCQ 1V8: 4u7 + 2 x 100n"
- note added: "VDDi: 2u2 (1-4.7 u)"
- note added: "e-MMC on bank 4A (1.8 V). Pull-ups to 1V8 (= VCCQ, same supply as the FPGA I/O as the data sheet requires)."

Commit message: LCSC numbers for all JLC parts; Y701 -> YXC OT322525MJBA4SL
- tools/set_lcsc.py: one table (value, footprint) -> LCSC, fills empty LCSC fields in the
  sheets; 312 symbols. JLC basic parts where available, cap voltages checked per rail,
  VCORE divider 0.1 % (no 0.5 % in stock). Board fields synced with add_parts.py.
- Y701: the SiT8924 has no JLC stock; now YXC OT322525MJBA4SL (C669088, 3225), EN tied
  to 1V8. R701/C701 moved 0.5 mm to clear its courtyard. Netlist change: Y701 pin 1 -> 1V8.
- Only U501 (Ti135) is left without LCSC (global sourcing / consigned).
- DRC: schematic parity 0.

Co-Authored-By: Claude Opus 5.5 <noreply@anthropic.com>
Parts:
- C1001, C1004: LCSC (none) -> C23733
- C1002, C1003, C1005, C1006: LCSC (none) -> C1525
- C1007: LCSC (none) -> C12530
- R1001: LCSC (none) -> C25077
- R1010, R1011, R1012, R1013, R1014, R1015, R1016, R1017, R1018, R1019, R1020: LCSC (none) -> C25792
Changed lines of the file:
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@@
 			)
 		)
+		(property "LCSC" "C25792"
+			(at 38.1 154.94 0)
+			(effects
+				(font
+					(size 1.27 1.27)
+				)
+				(hide yes)
+			)
+		)
 		(pin "1"
 		)
@@
 			)
 		)
+		(property "LCSC" "C25792"
+			(at 129.54 154.94 0)
+			(effects
+				(font
+					(size 1.27 1.27)
+				)
+				(hide yes)
+			)
+		)
 		(pin "1"
 		)
@@
 			)
 		)
+		(property "LCSC" "C1525"
+			(at 46.99 203.2 0)
+			(effects
+				(font
+					(size 1.27 1.27)
+				)
+				(hide yes)
+			)
+		)
 		(pin "1"
 		)
@@
 			)
 		)
+		(property "LCSC" "C23733"
+			(at 38.1 203.2 0)
+			(effects
+				(font
+					(size 1.27 1.27)
+				)
+				(hide yes)
+			)
+		)
 		(pin "1"
 		)
@@
 			)
 		)
+		(property "LCSC" "C25792"
+			(at 109.22 154.94 0)
+			(effects
+				(font
+					(size 1.27 1.27)
+				)
+				(hide yes)
+			)
+		)
 		(pin "1"
 		)
@@
 			)
 		)
+		(property "LCSC" "C1525"
+			(at 132.08 203.2 0)
+			(effects
+				(font
+					(size 1.27 1.27)
+				)
+				(hide yes)
+			)
+		)
 		(pin "1"
 		)
@@
 			)
 		)
+		(property "LCSC" "C25792"
+			(at 99.06 154.94 0)
+			(effects
+				(font
+					(size 1.27 1.27)
+				)
+				(hide yes)
+			)
+		)
 		(pin "1"
 		)
@@
 			)
 		)
+		(property "LCSC" "C25792"
+			(at 78.74 154.94 0)
+			(effects
+				(font
+					(size 1.27 1.27)
+				)
+				(hide yes)
+			)
+		)
 		(pin "1"
 		)
@@
 			)
 		)
+		(property "LCSC" "C25077"
+			(at 50.8 63.5 0)
+			(effects
+				(font
+					(size 1.27 1.27)
+				)
+				(hide yes)
+			)
+		)
 		(pin "1"
 		)
@@
 			)
 		)
+		(property "LCSC" "C25792"
+			(at 88.9 154.94 0)
+			(effects
+				(font
+					(size 1.27 1.27)
+				)
+				(hide yes)
+			)
+		)
 		(pin "1"
 		)
@@
 			)
 		)
+		(property "LCSC" "C12530"
+			(at 190.5 203.2 0)
+			(effects
+				(font
+					(size 1.27 1.27)
+				)
+				(hide yes)
+			)
+		)
 		(pin "1"
 		)
@@
 			)
 		)
+		(property "LCSC" "C1525"
+			(at 55.88 203.2 0)
+			(effects
+				(font
+					(size 1.27 1.27)
+				)
+				(hide yes)
+			)
+		)
 		(pin "1"
 		)
@@
 			)
 		)
+		(property "LCSC" "C25792"
+			(at 58.42 154.94 0)
+			(effects
+				(font
+					(size 1.27 1.27)
+				)
+				(hide yes)
+			)
+		)
 		(pin "1"
 		)
@@
 			)
 		)
+		(property "LCSC" "C25792"
+			(at 48.26 154.94 0)
+			(effects
+				(font
+					(size 1.27 1.27)
+				)
+				(hide yes)
+			)
+		)
 		(pin "1"
 		)
@@
 			)
 		)
+		(property "LCSC" "C23733"
+			(at 114.3 203.2 0)
+			(effects
+				(font
+					(size 1.27 1.27)
+				)
+				(hide yes)
+			)
+		)
 		(pin "1"
 		)
@@
 			)
 		)
+		(property "LCSC" "C1525"
+			(at 123.19 203.2 0)
+			(effects
+				(font
+					(size 1.27 1.27)
+				)
+				(hide yes)
+			)
+		)
 		(pin "1"
 		)
@@
 			)
 		)
+		(property "LCSC" "C25792"
+			(at 119.38 154.94 0)
+			(effects
+				(font
+					(size 1.27 1.27)
+				)
+				(hide yes)
+			)
+		)
 		(pin "1"
 		)
@@
 			)
 		)
+		(property "LCSC" "C25792"
+			(at 139.7 154.94 0)
+			(effects
+				(font
+					(size 1.27 1.27)
+				)
+				(hide yes)
+			)
+		)
 		(pin "1"
 		)
@@
 			)
 		)
+		(property "LCSC" "C25792"
+			(at 68.58 154.94 0)
+			(effects
+				(font
+					(size 1.27 1.27)
+				)
+				(hide yes)
+			)
+		)

Commit message: 3D models for the BGAs (U501, U801, U1001, U601)
KiCad's library has no model for any of them (the footprints pointed at
missing STEP files), so tools/gen_bga_3d.py writes simple VRML models
(body, pin-1 dot, balls) to lib/3dmodels, from datasheet dimensions:
Efinix N484 model, SK hynix 200-ball FBGA, Kioxia P-WFBGA153, ISSI 24-ball
TFBGA (H). Linked as ${KIPRJMOD}/../lib/3dmodels so the CI render finds them.

U501 and U1001 footprints copied into ti135_card.pretty (footprint fields
updated on board, schematic, symbol lib); the U501 copy carries the board's
pad-to-die delays, which clears its lib_footprint_mismatch. DRC parity clean.

Co-Authored-By: Claude Opus 5.5 <noreply@anthropic.com>
Parts:
- U1001: footprint Package_BGA:LFBGA-153_11.5x13mm_Layout14x14_P0.5mm -> ti135_card:LFBGA-153_11.5x13mm_Layout14x14_P0.5mm
Changed lines of the file:
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@@
 			)
 		)
-		(property "Footprint" "Package_BGA:LFBGA-153_11.5x13mm_Layout14x14_P0.5mm"
+		(property "Footprint" "ti135_card:LFBGA-153_11.5x13mm_Layout14x14_P0.5mm"
 			(at 190.5 101.6 0)
 			(hide yes)
