File: kicad/11_fpga_io.kicad_sch (KiCad schematic)
At the start: 1 part, among them U501 Ti135N484I3

Commit message: Phase 3 (half): checklist fixes in the schematic; board placement still to do
- R801 240R 0.1 % (RT0402BRD07240RL, C852660); SSU_N (L4) 10 k pull-up R622 to 1V8.
- Efinix decoupling table in full on sheet 05 (now A2): C5001-C5073 (0201 10n/1n/100n,
  0402 1u/4u7, 0805 10u/47u, 1206 100u).
- Each TLV62585 cell: 47u output cap and a 22p feed-forward cap across R1 (data sheet:
  feed-forward needed above 47 uF; user decision).
- build_schematic.sh fails on duplicate references (ERC misses them).
- tools/add_parts.py: add missing schematic parts to a routed board; tools/place_free.py
  (untested): nearest free B.Cu spot.
- kicad/ti135_card.kicad_pcb unchanged; placement in work/p3, see NEXT_SESSION.md.

Co-Authored-By: Claude Opus 5.5 <noreply@anthropic.com>
Connections:
- net fpga_ssu_n: now reaches U501.L4 (GPIOB_N_20_SSU_N_CLK6_N)
- no-connect marks 9 -> 8
Changed lines of the file:
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@@
 		)
 	)
-	(no_connect
-		(at 60.96 68.58)
+	(wire
+		(pts
+			(xy 60.96 68.58) (xy 55.88 68.58)
+		)
+		(stroke
+			(width 0)
+			(type default)
+		)
+	)
+	(hierarchical_label "fpga_ssu_n"
+		(shape passive)
+		(at 55.88 68.58 180)
+		(effects
+			(font
+				(size 1.27 1.27)
+			)
+			(justify right)
+		)
 	)
 	(wire

Commit message: 3D models for the BGAs (U501, U801, U1001, U601)
KiCad's library has no model for any of them (the footprints pointed at
missing STEP files), so tools/gen_bga_3d.py writes simple VRML models
(body, pin-1 dot, balls) to lib/3dmodels, from datasheet dimensions:
Efinix N484 model, SK hynix 200-ball FBGA, Kioxia P-WFBGA153, ISSI 24-ball
TFBGA (H). Linked as ${KIPRJMOD}/../lib/3dmodels so the CI render finds them.

U501 and U1001 footprints copied into ti135_card.pretty (footprint fields
updated on board, schematic, symbol lib); the U501 copy carries the board's
pad-to-die delays, which clears its lib_footprint_mismatch. DRC parity clean.

Co-Authored-By: Claude Opus 5.5 <noreply@anthropic.com>
Parts:
- U501: footprint Package_BGA:LFBGA-484_18x18mm_Layout22x22_P0.8mm -> ti135_card:LFBGA-484_18x18mm_Layout22x22_P0.8mm
Changed lines of the file:
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@@
 			)
 		)
-		(property "Footprint" "Package_BGA:LFBGA-484_18x18mm_Layout22x22_P0.8mm"
+		(property "Footprint" "ti135_card:LFBGA-484_18x18mm_Layout22x22_P0.8mm"
 			(at 317.5 66.04 0)
 			(hide yes)
@@
 			)
 		)
-		(property "Footprint" "Package_BGA:LFBGA-484_18x18mm_Layout22x22_P0.8mm"
+		(property "Footprint" "ti135_card:LFBGA-484_18x18mm_Layout22x22_P0.8mm"
 			(at 317.5 190.5 0)
 			(hide yes)
@@
 			)
 		)
-		(property "Footprint" "Package_BGA:LFBGA-484_18x18mm_Layout22x22_P0.8mm"
+		(property "Footprint" "ti135_card:LFBGA-484_18x18mm_Layout22x22_P0.8mm"
 			(at 101.6 66.04 0)
 			(hide yes)
@@
 			)
 		)
-		(property "Footprint" "Package_BGA:LFBGA-484_18x18mm_Layout22x22_P0.8mm"
+		(property "Footprint" "ti135_card:LFBGA-484_18x18mm_Layout22x22_P0.8mm"
 			(at 101.6 190.5 0)
 			(hide yes)
